File: thermometer.kicad_sch (KiCad schematic)
At the start: 3 parts, among them J1 Conn_01x07, U1 MCP9600-E_MX

Commit message: Add files via upload
Parts:
- removed J1: Conn_01x07, Connector_PinHeader_1.00mm:PinHeader_1x07_P1.00mm_Vertical, symbol Connector_Generic:Conn_01x07
- added J2: Conn_01x06, Connector_PinHeader_1.00mm:PinHeader_1x06_P1.00mm_Vertical, symbol Connector_Generic:Conn_01x06
Connections:
- net GND: now also U1.16 (ADDR), U1.21 (EXP), U1.22 (EXP), U1.23 (EXP), U1.24 (EXP), U1.25 (EXP), U1.26 (EXP), U1.27 (EXP), U1.28 (EXP), U1.29 (EXP), U1.30 (EXP)
- net ALERT_1: now reaches U1.11 (ALERT_1)
- net ALERT_1: now also J2.4 (Pin_4)
- net ALERT_2: now reaches U1.12 (ALERT_2)
- net ALERT_2: now also J2.3 (Pin_3)
- net ALERT_3: now reaches U1.14 (ALERT_3)
- net ALERT_3: now also J2.2 (Pin_2)
- net ALERT_4: now reaches U1.15 (ALERT_4)
- net ALERT_4: now also J2.1 (Pin_1)
- net SCL: now reaches U1.19 (SCL)
- net SCL: now also J2.6 (Pin_6)
- net SDA: now reaches U1.20 (SDA)
- net SDA: now also J2.5 (Pin_5)
